File: Eagle/fancontrollermegashield.sch (EAGLE design)
At the start: 27 parts, among them J1 FAN1, J2 MOLEX_47053-1000MOLEX_47053-1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, J3 POE HDR, J4 MOLEX_47053-1000MOLEX_47053-1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, J5 MOLEX_47053-1000MOLEX_47053-1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, J6 OLED, J7 TEMP1, J8 TEMP2

Commit message: Minor corrections
Connections:
- net POE_VIN: now also JP6.3
Other:
- note removed: "THIS IS THE WRONG HEADER - NEEDS TO BE FEMALE NOT MALE"
Changed lines of the file:
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@@
 <wire x1="180.34" y1="33.02" x2="180.34" y2="88.9" width="0.1524" layer="97" style="longdash"/>
 <wire x1="180.34" y1="88.9" x2="233.68" y2="88.9" width="0.1524" layer="97" style="longdash"/>
-<text x="48.26" y="78.74" size="1.778" layer="91">THIS IS THE WRONG HEADER - NEEDS TO BE FEMALE NOT MALE</text>
 <wire x1="40.64" y1="86.36" x2="111.76" y2="86.36" width="0.1524" layer="97" style="longdash"/>
 <wire x1="111.76" y1="86.36" x2="111.76" y2="180.34" width="0.1524" layer="97" style="longdash"/>
@@
 <label x="71.12" y="73.66" size="1.778" layer="95"/>
 </segment>
-</net>
+<segment>
+<pinref part="JP6" gate="G$1" pin="3"/>
+<wire x1="86.36" y1="104.14" x2="104.14" y2="104.14" width="0.1524" layer="91"/>
+<label x="101.6" y="104.14" size="1.778" layer="95"/>
+</segment>
+</net>
